File: kicadFiles/doddle60.kicad_pcb (KiCad board)
At the start: 2 copper layers, 283 x 94.2 mm, 183 parts, among them J1 TYPE-C-31-M12_13, J2 Conn_01x14, J3 Conn_ARM_JTAG_SWD_10, SW1 ESC, SW10 9, SW11 0, SW12 -_, SW13 +=, SW14 2U BKSP, SW15 TAB_150, SW16 Q, SW17 W, SW18 E, SW19 R, SW2 1, SW20 T, SW21 Y, SW22 U, SW23 I, SW24 O, SW25 P, SW26 [{, SW27 ]}, SW28 1U_RBKSP, SW29 CAPS_175, SW3 2, SW30 A, SW31 S, SW32 D, SW33 F, SW34 G, SW35 H, SW36 J, SW37 K, SW38 L, SW39 :;, SW4 3, SW40 @', SW41 ~~#, SW42 LSHIFT_125, SW43 |\, SW44 Z, SW45 X, SW46 C, SW47 V, SW48 B, SW49 N, SW5 4, SW50 M, SW51 <,, SW52 >., SW53 ?/, SW54 LCTRL_150, SW55 LGUI_100, SW56 LALT_150, SW57 SPACE_700, SW58 RALT_150, SW59 RGUI_100, SW6 5, SW60 RCTRL_150, SW61 LCTRL_125, SW62 LGUI_125, SW63 STEPPED_CAPS_125, SW64 1U LBKSP, SW65 ISO_Enter, SW66 LALT_125, SW67 SPACE_625, SW68 RALT_125, SW69 RGUI_125, SW7 6, SW70 FN_125, SW71 RCTRL_125, SW72 RSHIFT_275, SW8 7, SW9 8, U1 STM32F072-LQFP48, U2 USBLC6-2SC6, U3 MCP1700-3302E_SOT23

Commit message: Incorporate feedback from GeekHack IC
- There was a big feedback from the community on the GeekHack Interest Check thread (https://geekhack.org/index.php?topic=103057), mainly the lack of split right shift conpatibility and 2.25 left shift for US-ISO layouts. Hence both split right shift and 2.25U left shift were added.

- Some tweaks were made in the LDO area. Input and output resistors were added to discharge all the capacitors once the PCB is not energized. Also the value os CSO1 was changed from 100nF to 1uF for better voltage regulation.
Parts:
- added D63: 1N4148, acheron_Components:D_SOD-123, F.Cu at (89.0, 142.6)
- added RPU1: 1.5k, acheron_Components:R_SMD_1026, F.Cu at (330.7, 99.6)
- added RSI1: 100k, acheron_Components:R_SMD_1026, F.Cu at (311.5, 144.1)
- added RSO1: 100k, acheron_Components:R_SMD_1026, F.Cu at (322.6, 152.8)
- added SW73: LSHIFT_225, acheron_MX_SolderMask:MX225, F.Cu at (334.3, 148.5)
- added SW74: RSHIFT_175, acheron_MX_SolderMask:MX175, F.Cu at (105.7, 148.5)
- added SW75: FN_100, acheron_MX_SolderMask:MX100, F.Cu at (79.5, 148.5)
- CSO1: value 100n -> 1u
- moved D44 8.42 mm to (304.5, 141.4)
- moved D43 1.62 mm to (327.9, 141.4)
Connections:
- SW72 pad 1: Col14 -> Col13
Routing:
- net Row4: track 248.8 -> 281.2 mm
- net Col14: track 376.5 -> 358.6 mm
- net 3.3V: track 246.5 -> 260.0 mm
- net Col13: track 323.4 -> 335.9 mm
- net VBUS: track 31.4 -> 43.5 mm, vias 2 -> 3
- net Col1: track 185.9 -> 192.7 mm
- net Net-(D63-Pad2): track 0.00 -> 6.45 mm
- net DBus-: track 15.8 -> 21.0 mm
- net 5V: track 97.7 -> 100.3 mm
- net Net-(D44-Pad2): track 6.40 -> 4.04 mm
- net Net-(D43-Pad2): track 5.62 -> 3.66 mm
- net Row1: track 570.1 -> 572.0 mm
- net Net-(D62-Pad2): track 15.4 -> 16.7 mm

Commit message: Run DRC
- DRC was ran and issues solved
Parts:
- moved D55 4.76 mm to (333.1, 161.6)
- moved D54 4.63 mm to (349.5, 160.4)
Routing:
- net BOOT0: track 118.0 -> 126.3 mm
- net NRST: track 154.3 -> 162.4 mm
- net Net-(D55-Pad2): track 7.64 -> 12.4 mm
- net Row5: track 385.4 -> 381.6 mm
- net Net-(D54-Pad2): track 2.67 -> 6.35 mm
- net 3.3V: track 260.0 -> 263.6 mm
- net SWDIO: track 102.7 -> 104.1 mm
- net SWCLK: track 97.9 -> 99.3 mm

Commit message: Update KLE and renders
Routing:
- net Col1: track 192.7 -> 195.0 mm
Changed lines of the file:
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@@
     (thickness 1.6)
     (drawings 136)
-    (tracks 1584)
+    (tracks 1585)
     (zones 0)
     (modules 190)
@@
   (segment (start 335.76225 139.391065) (end 331.72995 143.423365) (width 0.5) (layer B.Cu) (net 10))
   (segment (start 335.76225 131.993125) (end 335.76225 138.343125) (width 0.5) (layer B.Cu) (net 10))
+  (segment (start 338.87373 162.473445) (end 341.255 162.473445) (width 0.254) (layer F.Cu) (net 10))
   (segment (start 330.93617 88.813125) (end 329.63625 88.813125) (width 1) (layer F.Cu) (net 11))
   (segment (start 329.63625 88.813125) (end 329.17625 88.353125) (width 1) (layer F.Cu) (net 11))

Commit message: Implement filters, TVS and LED
- The pi filter for VDD and GNDD was implemented; the common mode choke
added to the schematic on the last commit was deemed unnecessary and
thence removed

- The TVS and choke for VBUS-5V was implemented;

- The common mode choke for USB data lines was added
Parts:
- added CB10: 1µ, Capacitor_SMD:C_0805_2012Metric, F.Cu at (321.9, 129.2)
- added CB9: 1µ, Capacitor_SMD:C_0805_2012Metric, F.Cu at (321.9, 134.8)
- added DL1: 19-217/R6C-AL1M2VY/3T, LED_SMD:LED_0603_1608Metric, F.Cu at (307.6, 141.6)
- added G1: Doddle60Logo, doddle60Graphics:doddle60Logo, B.Cu at (250.0, 167.2)
- added G4: Doddle60Label, doddle60Graphics:doddle60Label, F.Cu at (250.9, 167.6)
- added L2: MGFL1608F1R0MT-LF, Inductor_SMD:L_0603_1608Metric, F.Cu at (347.8, 98.0)
- added RL1: 620R, acheron_Components:R_SMD_1026, F.Cu at (311.5, 140.4)
- added RVDD1: 0R 1%, acheron_Components:R_SMD_1026, F.Cu at (325.7, 131.9)
- CB1: value 1uF -> 1µ
- CB2: value 10n -> 100n
- CB4, CB6: value 4.7uF -> 1µ
- DF1: value RB060M-60TR -> SMF9.0CA; footprint acheron_Components:D_SOD-123 -> acheron_Components:D_SOD-123_Bidirectional
- DRST1: value 1N4148 -> B0520LW
- DS1: value 1N4148 -> RB060M-60TR
- DSH1: value 1N4007 -> RB060M-60TR
- F1: value Polyfuse -> 1A trip PTC
- L1: value Doddle60Logo -> ACM2012-900-2P-T002; footprint doddle60Graphics:doddle60Logo -> acheron_Components:ACM2012-2P; moved to F.Cu
- L4: value Doddle60Label -> CMI322513U1R0KT; footprint doddle60Graphics:doddle60Label -> Inductor_SMD:L_1210_3225Metric
- moved L1 109.1 mm to (336.0, 100.8), turned to 270 degrees
- moved L4 79.4 mm to (321.9, 132.0)
- moved D30 16.1 mm to (306.3, 134.2)
- moved D15 3.62 mm to (331.9, 105.0), turned to 0 degrees
- moved D1 1.74 mm to (351.2, 95.2)
- moved CB8 0.40 mm to (321.9, 114.6)
- moved CB7 0.27 mm to (321.3, 116.4), turned to 90 degrees
- renumbered L2 to G2, L3 to G3, L5 to G5
Connections:
- CB1 pad 1: GND -> GNDD
- CB1 pad 2: 3.3V -> VDD
- CB2 pad 1: GND -> GNDD
- CB2 pad 2: 3.3V -> VDD
- CB3 pad 1: GND -> GNDD
- CB3 pad 2: 3.3V -> VDD
- CB4 pad 1: GND -> GNDD
- CB4 pad 2: 3.3V -> VDD
- CB5 pad 1: GND -> GNDD
- CB5 pad 2: 3.3V -> VDD
- CB6 pad 1: GND -> GNDD
- CB6 pad 2: 3.3V -> VDD
- CB7 pad 1: 3.3V -> VDD
- CB7 pad 2: GND -> GNDD
- CB8 pad 1: GND -> GNDD
- CB8 pad 2: 3.3V -> VDD
- DF1 pad 1: 5V -> Net-(DF1-Pad1)
- F1 pad 1: 5V -> Net-(DF1-Pad1)
- J1 pad A6: DBus- -> DBus+
- J1 pad A7: DBus+ -> DBus-
- J1 pad B6: DBus- -> DBus+
- J1 pad B7: DBus+ -> DBus-
- RPU1 pad 2: DBus- -> DBus+
- U1 pad 1: 3.3V -> VDD
- U1 pad 23: GND -> GNDD
- U1 pad 24: 3.3V -> VDD
- U1 pad 35: GND -> GNDD
- U1 pad 36: 3.3V -> VDD
- U1 pad 47: GND -> GNDD
- U1 pad 48: 3.3V -> VDD
- U1 pad 8: GND -> GNDD
- U1 pad 9: 3.3V -> VDD
- U2 pad 1: D- -> Net-(L1-Pad2)
- U2 pad 3: D+ -> Net-(L1-Pad1)
- U2 pad 4: DBus+ -> DBus-
- U2 pad 6: DBus- -> DBus+
Routing:
- net VDD: track 0.00 -> 69.0 mm, vias 0 -> 6
- net 3.3V: track 263.6 -> 195.1 mm, vias 5 -> 2
- net D+: track 65.3 -> 46.7 mm
- net GNDD: track 0.00 -> 16.3 mm, vias 0 -> 2
- net D-: track 56.8 -> 44.7 mm
- net Col1: track 195.0 -> 183.0 mm
- net Col2: track 127.2 -> 138.7 mm
- net Net-(D30-Pad2): track 9.88 -> 16.6 mm
- net Row2: track 278.6 -> 272.0 mm
- net Net-(DF1-Pad1): track 0.00 -> 6.38 mm
- net DBus-: track 21.0 -> 15.8 mm, vias 2 -> 0
- net DBus+: track 15.8 -> 21.0 mm, vias 0 -> 2
- net VBUS: track 43.5 -> 48.7 mm
- net SWDIO: track 104.1 -> 99.2 mm
- net 5V: track 100.3 -> 95.5 mm
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- added copper zone on F.Cu, net GNDD
- added copper zone on B.Cu, net VDD
Other:
- net class Default: clearance 0.127 -> 0.1524
- rule trace_clearance: 0.127 -> 0.1524

Commit message: Add layout indicator silkscreen
Parts:
- moved RSO1 10.6 mm to (332.6, 156.3)
Routing:
- net 3.3V: track 195.1 -> 187.5 mm
Other:
- board text added: "1.00 FN"
- board text added: "1.00 LGUI"
- board text added: "1.00 RGUI"
- board text added: "1.00 SPLIT LSHFT"
- board text added: "1.25 FN"
- board text added: "1.25 LALT"
- board text added: "1.25 LCTRL"
- board text added: "1.25 LGUI"
- board text added: "1.25 LSHIFT"
- board text added: "1.25 RALT"
- board text added: "1.25 RCTRL"
- board text added: "1.25 RGUI"
- board text added: "1.50 LALT"
- board text added: "1.50 LCTRL"
- board text added: "1.50 RALT"
- board text added: "1.50 RCTRL"
- board text added: "1.75 RSHIFT"
- board text added: "1U BKSP"
- board text added: "2.25 LSHIFT"
- board text added: "2.75 RSHIFT"
- board text added: "2U BKSP"
- board text added: "6.25U SPACE"
- board text added: "7U SPACE"
