File: kicadFiles/doddle60.kicad_pcb (KiCad board)
At the start: 2 copper layers, 283 x 94.2 mm, 198 parts, among them J1 TYPE-C-31-M12_13, J2 Conn_01x14, J3 Conn_ARM_JTAG_SWD_10, SW1 ESC, SW10 9, SW11 0, SW12 -_, SW13 +=, SW14 2U BKSP, SW15 TAB_150, SW16 Q, SW17 W, SW18 E, SW19 R, SW2 1, SW20 T, SW21 Y, SW22 U, SW23 I, SW24 O, SW25 P, SW26 [{, SW27 ]}, SW28 1U_RBKSP, SW29 CAPS_175, SW3 2, SW30 A, SW31 S, SW32 D, SW33 F, SW34 G, SW35 H, SW36 J, SW37 K, SW38 L, SW39 :;, SW4 3, SW40 @', SW41 ~~#, SW42 LSHIFT_125, SW43 |\, SW44 Z, SW45 X, SW46 C, SW47 V, SW48 B, SW49 N, SW5 4, SW50 M, SW51 <,, SW52 >., SW53 ?/, SW54 LCTRL_150, SW55 LGUI_100, SW56 LALT_150, SW57 SPACE_700, SW58 RALT_150, SW59 RGUI_100, SW6 5, SW60 RCTRL_150, SW61 LCTRL_125, SW62 LGUI_125, SW63 STEPPED_CAPS_125, SW64 1U LBKSP, SW65 ISO_Enter, SW66 LALT_125, SW67 SPACE_625, SW68 RALT_125, SW69 RGUI_125, SW7 6, SW70 FN_125, SW71 RCTRL_125, SW72 RSHIFT_275, SW73 LSHIFT_225, SW74 RSHIFT_175, SW75 FN_100, SW8 7, SW9 8, U1 STM32F072-LQFP48, U2 USBLC6-2SC6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

Commit message: Update renders
Parts:
- CSI1: value 100n -> 1µ
- CSO1: value 1u -> 1µ
- RVDD1: value 0R 1% -> R010 1%
- renumbered L4 to L3
Other:
- net class Default: clearance 0.1524 -> 0.127
- rule trace_clearance: 0.1524 -> 0.127
Changed lines of the file:
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@@
   (page A3)
   (title_block
-    (title ArcticPCB)
-    (date 2019-11-04)
+    (title Doddle60)
+    (date 2019-11-11)
     (rev pre-Alpha)
-    (comment 1 "Designed by Gondolindrim in partnership with ArcticFox")
-    (comment 2 "Project page: http://github.com/Gondolindrim/ArcticPCB")
+    (company "Designed by Gondolindrim")
+    (comment 1 "In partnership with Jae@TopClack")
+    (comment 2 "Project page: http://github.com/Gondolindrim/Doddle60")
     (comment 3 "Doddle60: an ISO minimum layout, 60% custom keyboard PCB")
   )
@@
     (user_trace_width 0.5)
     (user_trace_width 1)
-    (trace_clearance 0.1524)
+    (trace_clearance 0.127)
     (zone_clearance 0.1524)
     (zone_45_only no)
@@
       (drillshape 0)
       (scaleselection 1)
-      (outputdirectory "../doddleGerbers"))
+      (outputdirectory "../preAlpha/"))
   )
   (net 0 "")
@@
   (net 126 "Net-(DL1-Pad2)")
   (net_class Default "This is the default net class."
-    (clearance 0.1524)
+    (clearance 0.127)
     (trace_width 0.254)
     (via_dia 0.8)
@@
     (add_net D-)
   )
+  (module acheron_Components:ACM2012-2P (layer F.Cu)
+    (at 335.97625 100.751125 270)
+    (clearance 0.1524)
+    (fp_text reference L1 (at 0 -1.5 90) (layer F.SilkS)
+      (effects (font (size 0.6 0.6) (thickness 0.12)))
+    )
+    (fp_text value ACM2012-900-2P-T002 (at 1.778 -0.04) (layer F.Fab)
+      (effects (font (size 0.2032 0.2032) (thickness 0.0508)))
+    )
+    (fp_line (start -1.4 0.8) (end -1.4 -0.8) (layer F.CrtYd) (width 0.05))
+    (fp_line (start 1.4 0.8) (end -1.4 0.8) (layer F.CrtYd) (width 0.05))
+    (fp_line (start 1.4 -0.8) (end 1.4 0.8) (layer F.CrtYd) (width 0.05))
+    (fp_line (start -1.4 -0.8) (end 1.4 -0.8) (layer F.CrtYd) (width 0.05))
+    (fp_poly (pts (xy -0.94 -1) (xy -1.24 -1.3) (xy -0.64 -1.3)) (layer F.SilkS) (width 0.1))
+    (fp_line (start -1.4 -0.8) (end 1.4 -0.8) (layer F.Fab) (width 0.0762))
+    (fp_line (start 1.4 -0.8) (end 1.4 0.8) (layer F.Fab) (width 0.0762))
+    (fp_line (start 1.4 0.8) (end -1.4 0.8) (layer F.Fab) (width 0.0762))
+    (fp_line (start -1.4 0.8) (end -1.4 -0.8) (layer F.Fab) (width 0.0762))
+    (fp_line (start -1.4 -0.1) (end -0.4 -0.1) (layer F.Fab) (width 0.0762))
+    (fp_line (start -0.4 -0.8) (end -0.4 -0.1) (layer F.Fab) (width 0.0762))
+    (fp_text user 1 (at -0.9 -0.45 90) (layer F.Fab)
+      (effects (font (size 0.381 0.381) (thickness 0.09525)))
+    )
+    (pad 3 smd rect (at 0.925 0.5 270) (size 0.75 0.4) (layers F.Cu F.Paste F.Mask)
+      (net 94 D+))
+    (pad 2 smd rect (at -0.925 0.5 270) (size 0.75 0.4) (layers F.Cu F.Paste F.Mask)
+      (net 125 "Net-(L1-Pad2)"))
+    (pad 1 smd roundrect (at -0.925 -0.5 270) (size 0.75 0.4) (layers F.Cu F.Paste F.Mask) (roundrect_rratio 0.25)
+      (net 124 "Net-(L1-Pad1)"))
+    (pad 4 smd rect (at 0.925 -0.5 270) (size 0.75 0.4) (layers F.Cu F.Paste F.Mask)
+      (net 95 D-))
+    (model ${KIPRJMOD}/AcheronLibrary/3d_models/ACM2012-2P.STEP
+      (offset (xyz 0 0 1.26))
+      (scale (xyz 1 1 1))
+      (rotate (xyz 90 0 0))
+    )
+  )
   (module acheron_Components:R_SMD_1026 (layer F.Cu)
     (at 325.72925 131.866125 270)
@@
       (effects (font (size 0.635 0.635) (thickness 0.127)))
     )
-    (fp_text value "0R 1%" (at 0 -1.397 90) (layer F.Fab)
+    (fp_text value "R010 1%" (at 0 -1.397 90) (layer F.Fab)
       (effects (font (size 0.6 0.6) (thickness 0.1)))
     )
@@
     (tags inductor)
     (attr smd)
-    (fp_text reference L4 (at -3.048 0 90) (layer F.SilkS)
+    (fp_text reference L3 (at -3.048 0 90) (layer F.SilkS)
       (effects (font (size 0.635 0.635) (thickness 0.15875)))
     )
@@
     )
   )
-  (module acheron_Components:ACM2012-2P (layer F.Cu)
-    (at 335.97625 100.751125 270)
-    (clearance 0.1524)
-    (fp_text reference L1 (at 0 -1.5 270) (layer F.SilkS)
-      (effects (font (size 0.6 0.6) (thickness 0.12)))
-    )
-    (fp_text value ACM2012-900-2P-T002 (at 1.778 -0.04) (layer F.Fab)
-      (effects (font (size 0.2032 0.2032) (thickness 0.0508)))
-    )
-    (fp_line (start -1.4 0.8) (end -1.4 -0.8) (layer F.CrtYd) (width 0.05))
-    (fp_line (start 1.4 0.8) (end -1.4 0.8) (layer F.CrtYd) (width 0.05))
-    (fp_line (start 1.4 -0.8) (end 1.4 0.8) (layer F.CrtYd) (width 0.05))
-    (fp_line (start -1.4 -0.8) (end 1.4 -0.8) (layer F.CrtYd) (width 0.05))
-    (fp_poly (pts (xy -0.94 -1) (xy -1.24 -1.3) (xy -0.64 -1.3)) (layer F.SilkS) (width 0.1))
-    (pad 3 smd rect (at 0.925 0.5 270) (size 0.75 0.4) (layers F.Cu F.Paste F.Mask)
-      (net 94 D+))
-    (pad 2 smd rect (at -0.925 0.5 270) (size 0.75 0.4) (layers F.Cu F.Paste F.Mask)
-      (net 125 "Net-(L1-Pad2)"))
-    (pad 1 smd roundrect (at -0.925 -0.5 270) (size 0.75 0.4) (layers F.Cu F.Paste F.Mask) (roundrect_rratio 0.25)
-      (net 124 "Net-(L1-Pad1)"))
-    (pad 4 smd rect (at 0.925 -0.5 270) (size 0.75 0.4) (layers F.Cu F.Paste F.Mask)
-      (net 95 D-))
-    (model ${KIPRJMOD}/AcheronLibrary/3d_models/ACM2012-2P.STEP
-      (offset (xyz 0 0 1.26))
-      (scale (xyz 1 1 1))
-      (rotate (xyz 90 0 0))
-    )
-  )
   (module acheron_Components:LQFP-48_7x7mm_P0.5mm (layer F.Cu)
     (at 327.12617 119.928245)
@@
       (effects (font (size 0.6 0.6) (thickness 0.12)))
     )
-    (fp_text value 100n (at 0 -1.368) (layer F.Fab)
+    (fp_text value 1µ (at 0 -1.368) (layer F.Fab)
       (effects (font (size 0.5 0.5) (thickness 0.1)))
     )
@@
       (effects (font (size 0.6 0.6) (thickness 0.12)))
     )
-    (fp_text value 1u (at 0 1.119) (layer F.Fab)
+    (fp_text value 1µ (at 0 1.119) (layer F.Fab)
       (effects (font (size 0.5 0.5) (thickness 0.1)))
     )
@@
       (effects (font (size 0.6 0.6) (thickness 0.12)))
     )
-    (fp_text value 100n (at -2.036 0.088 90) (layer F.Fab)
+    (fp_text value 100n (at 2.282 0.088 90) (layer F.Fab)
       (effects (font (size 0.5 0.5) (thickness 0.1)))
     )
