File: kicadFiles/doddle60.sch (KiCad schematic (older format))
At the start: 183 parts, among them J1 TYPE-C-31-M12_13, J2 Conn_01x14, J3 Conn_ARM_JTAG_SWD_10, SW1 ESC, SW10 9, SW11 0, SW12 -_, SW13 +=, SW14 2U BKSP, SW15 TAB_150, SW16 Q, SW17 W, SW18 E, SW19 R, SW2 1, SW20 T, SW21 Y, SW22 U, SW23 I, SW24 O, SW25 P, SW26 [{, SW27 ]}, SW28 1U_RBKSP, SW29 CAPS_175, SW3 2, SW30 A, SW31 S, SW32 D, SW33 F, SW34 G, SW35 H, SW36 J, SW37 K, SW38 L, SW39 :;, SW4 3, SW40 @', SW41 ~~#, SW42 LSHIFT_125, SW43 |\\, SW44 Z, SW45 X, SW46 C, SW47 V, SW48 B, SW49 N, SW5 4, SW50 M, SW51 <,, SW52 >., SW53 ?/, SW54 LCTRL_150, SW55 LGUI_100, SW56 LALT_150, SW57 SPACE_700, SW58 RALT_150, SW59 RGUI_100, SW6 5, SW60 RCTRL_150, SW61 LCTRL_125, SW62 LGUI_125, SW63 STEPPED_CAPS_125, SW64 1U LBKSP, SW65 ISO_Enter, SW66 LALT_125, SW67 SPACE_625, SW68 RALT_125, SW69 RGUI_125, SW7 6, SW70 FN_125, SW71 RCTRL_125, SW72 RSHIFT_275, SW8 7, SW9 8, U1 STM32F072-LQFP48, U2 USBLC6-2SC6, U3 MCP1700-3302E_SOT23

Commit message: Incorporate feedback from GeekHack IC
- There was a big feedback from the community on the GeekHack Interest Check thread (https://geekhack.org/index.php?topic=103057), mainly the lack of split right shift conpatibility and 2.25 left shift for US-ISO layouts. Hence both split right shift and 2.25U left shift were added.

- Some tweaks were made in the LDO area. Input and output resistors were added to discharge all the capacitors once the PCB is not energized. Also the value os CSO1 was changed from 100nF to 1uF for better voltage regulation.
Parts:
- added D63: 1N4148, acheron_Components:D_SOD-123, symbol Device:D
- added RPU1: 1.5k, acheron_Components:R_SMD_1026, symbol Device:R_Small
- added RSI1, RSO1: 100k, acheron_Components:R_SMD_1026, symbol Device:R_Small
- added SW73: LSHIFT_225, acheron_MX_SolderMask:MX225, symbol acheronSymbols:MXSwitch
- added SW74: RSHIFT_175, acheron_MX_SolderMask:MX175, symbol acheronSymbols:MXSwitch
- added SW75: FN_100, acheron_MX_SolderMask:MX100, symbol acheronSymbols:MXSwitch
- CSO1: value 100n -> 1u
Connections:
- net 3.3V: now also RSO1.1
- net 5V: now also RSI1.1
- net Col1: now also SW73.1 (Col)
- net Col13: now also SW72.1 (Col), SW74.1 (Col)
- net Col14: now also SW75.1 (Col); no longer SW72.1 (Col)
- net DBus-: now also RPU1.2
- net GND: now also RSI1.2, RSO1.2
- net Row4: now also D63.1 (K)
- net VBUS: now also RPU1.1
- net at D62.2 (A), SW72.2 (Row): now also SW74.2 (Row)
- net at D42.2 (A), SW42.2 (Row): now also SW73.2 (Row)
- new net: D63.2 (A), SW75.2 (Row)
Other:
- moved on the sheet: CSI1, CSO1, D62, SW72

Commit message: Update KLE and renders
Parts:
- added L?: MGFL1608F1R0MT-LF, Inductor_SMD:L_0603_1608Metric, symbol Device:L_Core_Ferrite
- added L? (x2): L_Core_Ferrite_Coupled_1423, symbol acheronSymbols:L_Core_Ferrite_Coupled_1423
- DF1: value RB060M-60TR -> SMF9.0CA; footprint acheron_Components:D_SOD-123 -> acheron_Components:D_SOD-123_Bidirectional; symbol Device:D_Schottky -> Device:D_TVS
- DRST1: value 1N4148 -> B0520LW
- DS1: value 1N4148 -> RB060M-60TR
- DSH1: value 1N4007 -> RB060M-60TR
- F1: value Polyfuse -> 1A trip PTC
Connections:
- net 5V: now also L?.2; no longer DF1.1 (K), F1.1
- new net: DF1.1 (A1), F1.1, L?.1
Other:
- moved on the sheet: CSI1, CSO1, DS1, RSI1, RSO1, U3

Commit message: Add TVS, diff impedance, pi filter
- A TVS diode was added to the VBUS power rail for more stability and voltage clamping;

- A differential mode choke was added to the data lines;

- A pi filter with a differential mode choke was added to the MCU power circuit for isolation and stability
Parts:
- added CB? (x2): 1u, Capacitor_SMD:C_0402_1005Metric, symbol Device:C_Small
- added L?: CMI201209VR33KT, Inductor_SMD:L_0805_2012Metric, symbol Device:L_Core_Ferrite
- CB2: value 10n -> 100n
- CB4, CB6: value 4.7uF -> 1u
- L?: value L_Core_Ferrite_Coupled_1423 -> ACM2012-900-2P-T002; footprint (none) -> acheron_Components:ACM2012-2P
- L?: value L_Core_Ferrite_Coupled_1423 -> EXC14CE900U; footprint (none) -> acheron_Components:EXC14CG-CE
- renumbered L1 to G1, L2 to G2, L3 to G3, L4 to G4, L5 to G5
Connections:
- net 3.3V: now also L?.1; no longer CB1.2, CB2.2, CB3.2, CB4.2, CB5.2, CB6.2, CB7.1, CB8.2, U1.1 (VBAT), U1.24 (VDD), U1.36 (VDDIO2), U1.48 (VDD), U1.9 (VDDA)
- net DBus+: now also L?.3; no longer J1.A7 (D-), J1.B7 (D-)
- net DBus-: now also L?.4; no longer J1.A6 (D+), J1.B6 (D+), RPU1.2
- net GND: now also L?.2; no longer CB1.1, CB2.1, CB3.1, CB4.1, CB5.1, CB6.1, CB7.2, CB8.1, U1.23 (VSS), U1.35 (VSS), U1.47 (VSS), U1.8 (VSSA)
- net GNDD: now reaches L?.3
- net GNDD: now also CB1.1, CB2.1, CB3.1, CB4.1, CB5.1, CB6.1, CB7.2, CB8.1, U1.23 (VSS), U1.35 (VSS), U1.47 (VSS), U1.8 (VSSA), CB?.1, CB?.1
- net at L?.4: now also CB?.2, L?.1
- net at L?.1: now also J1.A7 (D-), J1.B7 (D-)
- net at L?.2: now also J1.A6 (D+), J1.B6 (D+), RPU1.2
- new net VDD: CB1.2, CB2.2, CB3.2, CB4.2, CB5.2, CB6.2, CB7.1, CB8.2, CB?.2, L?.2, U1.1 (VBAT), U1.24 (VDD), U1.36 (VDDIO2), U1.48 (VDD), U1.9 (VDDA)
Other:
- moved on the sheet: CB1, CB2, CB3, CB4, CB5, CB6, CB7, CB8, CSH1, J1, L?, RCC1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

Commit message: Implement filters, TVS and LED
- The pi filter for VDD and GNDD was implemented; the common mode choke
added to the schematic on the last commit was deemed unnecessary and
thence removed

- The TVS and choke for VBUS-5V was implemented;

- The common mode choke for USB data lines was added
Parts:
- removed L?: ACM2012-900-2P-T002, acheron_Components:ACM2012-2P, symbol acheronSymbols:L_Core_Ferrite_Coupled_1423
- removed L?: EXC14CE900U, acheron_Components:EXC14CG-CE, symbol acheronSymbols:L_Core_Ferrite_Coupled_1423
- added DL1: 19-217/R6C-AL1M2VY/3T, LED_SMD:LED_0603_1608Metric, symbol Device:LED_Small
- added L1: ACM2012-900-2P-T002, acheron_Components:ACM2012-2P, symbol acheronSymbols:L_Core_Ferrite_Coupled_1423
- added RL1: 620R, acheron_Components:R_SMD_1026, symbol Device:R_Small
- added RVDD1: R010 1%, acheron_Components:R_SMD_1026, symbol Device:R_Small
- CB1: value 1uF -> 1µ
- CB10, CB9: renamed from CB?; value 1u -> 1µ; footprint Capacitor_SMD:C_0402_1005Metric -> Capacitor_SMD:C_0805_2012Metric
- CB4, CB6: value 1u -> 1µ
- DRST1, DS1, DSH1: symbol Device:D -> Device:D_Schottky
- L4: renamed from L?; value CMI201209VR33KT -> CMI322513U1R0KT; footprint Inductor_SMD:L_0805_2012Metric -> Inductor_SMD:L_1210_3225Metric
- gave numbers to parts that had none: 1
Connections:
- net 3.3V: now also CB9.2, L4.1
- net 5V: now also RL1.1
- net D+: now also L1.3; no longer U2.3 (IO2)
- net D-: now also L1.4; no longer U2.1 (IO1)
- net DBus+: now also J1.A6 (D+), J1.B6 (D+), RPU1.2, U2.6 (IO1); no longer U2.4 (IO2)
- net DBus-: now also J1.A7 (D-), J1.B7 (D-), U2.4 (IO2); no longer U2.6 (IO1)
- net GND: now also CB9.1, DL1.1 (K), RVDD1.2
- net GNDD: now also RVDD1.1; no longer CB9.1
- new net: L1.2, U2.1 (IO1)
- new net: L1.1, U2.3 (IO2)
- new net: DL1.2 (A), RL1.2

Commit message: Update renders
Parts:
- CSI1: value 100n -> 1µ
- CSO1: value 1u -> 1µ
- renumbered L4 to L3
Changed lines of the file:
@@
 Sheet 1 1
 Title "Doddle60"
-Date "2019-11-04"
+Date "2019-11-11"
 Rev "pre-Alpha"
 Comp "Designed by Gondolindrim"
-Comment1 ""
+Comment1 "In partnership with Jae@TopClack"
 Comment2 ""
 Comment3 ""
@@
 P 10150 15125
 F 0 "CSI1" V 10250 15125 39  0000 C CNN
-F 1 "100n" V 10050 15125 31  0000 C CNN
+F 1 "1µ" V 10050 15125 31  0000 C CNN
 F 2 "Capacitor_SMD:C_0805_2012Metric_Pad1.15x1.40mm_HandSolder" H 10150 15125 50  0001 C CNN
 F 3 "~" H 10150 15125 50  0001 C CNN
@@
 P 10850 15125
 F 0 "CSO1" H 10975 15200 39  0000 C CNN
-F 1 "1u" H 10950 15275 39  0000 C CNN
+F 1 "1µ" H 10950 15275 39  0000 C CNN
 F 2 "Capacitor_SMD:C_0805_2012Metric_Pad1.15x1.40mm_HandSolder" H 10850 15125 50  0001 C CNN
 F 3 "~" H 10850 15125 50  0001 C CNN
@@
 	13500 9575 13575 9575
 $Comp
-L Device:L_Core_Ferrite L4
+L Device:L_Core_Ferrite L3
 U 1 1 5F75AC01
 P 13850 9575
-F 0 "L4" V 14045 9575 50  0000 C CNN
+F 0 "L3" V 14045 9575 50  0000 C CNN
 F 1 "CMI322513U1R0KT" V 13968 9575 30  0000 C CNN
 F 2 "Inductor_SMD:L_1210_3225Metric" H 13850 9575 50  0001 C CNN
